File: yuki_pcb/yuki_pcb.kicad_pcb (KiCad board)
At the start: 2 copper layers, 139.5 x 94.6 mm, 28 parts, among them J1 TRRS, K00 KEYSW, K01 KEYSW, K02 KEYSW, K03 KEYSW, K04 KEYSW, K05 KEYSW, K10 KEYSW, K11 KEYSW, K12 KEYSW, K13 KEYSW, K14 KEYSW, K15 KEYSW, K20 KEYSW, K21 KEYSW, K22 KEYSW, K23 KEYSW, K24 KEYSW, K25 KEYSW, K30 KEYSW, K31 KEYSW, K32 KEYSW, K33 KEYSW, U1 YAAJ_WeAct_BlackPill_Part_Like

Commit message: v0.2
Routing:
- net /k33: track 70.8 -> 70.0 mm
Other:
- board text removed: "DS1"
