File: yuki_pcb/yuki_pcb.kicad_sch (KiCad schematic)
At the start: 25 parts, among them J1 TRRS, K00 KEYSW, K01 KEYSW, K02 KEYSW, K03 KEYSW, K04 KEYSW, K05 KEYSW, K10 KEYSW, K11 KEYSW, K12 KEYSW, K13 KEYSW, K14 KEYSW, K15 KEYSW, K20 KEYSW, K21 KEYSW, K22 KEYSW, K23 KEYSW, K24 KEYSW, K25 KEYSW, K30 KEYSW, K31 KEYSW, K32 KEYSW, K33 KEYSW, U1 YAAJ_WeAct_BlackPill_Part_Like

Commit message: v0.2 with Choc switches!
Parts:
- K00, K01, K02, K03, K04, K05, K10, K11, K12, K13, K14, K15, K20, K21, K22, K23, K24, K25, K30, K31, K32, K33: footprint YUKI:CherryMX_rev -> YUKI:Kailh_Choc_PG1350_rev
Changed lines of the file:
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@@
 	(label "k23"
 		(at 82.55 73.66 0)
-		(fields_autoplaced yes)
 		(effects
 			(font
@@
 	(label "SCL"
 		(at 64.77 138.43 0)
-		(fields_autoplaced yes)
 		(effects
 			(font
@@
 	(label "k32"
 		(at 207.01 104.14 0)
-		(fields_autoplaced yes)
 		(effects
 			(font
@@
 	(label "k11"
 		(at 129.54 73.66 0)
-		(fields_autoplaced yes)
 		(effects
 			(font
@@
 	(label "k15"
 		(at 29.21 68.58 0)
-		(fields_autoplaced yes)
 		(effects
 			(font
@@
 	(label "k01"
 		(at 29.21 63.5 0)
-		(fields_autoplaced yes)
 		(effects
 			(font
@@
 	(label "k24"
 		(at 82.55 76.2 0)
-		(fields_autoplaced yes)
 		(effects
 			(font
@@
 	(label "k13"
 		(at 29.21 81.28 0)
-		(fields_autoplaced yes)
 		(effects
 			(font
@@
 	(label "k12"
 		(at 154.94 73.66 0)
-		(fields_autoplaced yes)
 		(effects
 			(font
@@
 	(label "k14"
 		(at 29.21 76.2 0)
-		(fields_autoplaced yes)
 		(effects
 			(font
@@
 	(label "k31"
 		(at 82.55 83.82 0)
-		(fields_autoplaced yes)
 		(effects
 			(font
@@
 	(label "k33"
 		(at 82.55 88.9 0)
-		(fields_autoplaced yes)
 		(effects
 			(font
@@
 	(label "RX"
 		(at 29.21 88.9 0)
-		(fields_autoplaced yes)
 		(effects
 			(font
@@
 	(label "k12"
 		(at 29.21 83.82 0)
-		(fields_autoplaced yes)
 		(effects
 			(font
@@
 	(label "k25"
 		(at 82.55 78.74 0)
-		(fields_autoplaced yes)
 		(effects
 			(font
@@
 	(label "k22"
 		(at 82.55 71.12 0)
-		(fields_autoplaced yes)
 		(effects
 			(font
@@
 	(label "k20"
 		(at 82.55 66.04 0)
-		(fields_autoplaced yes)
 		(effects
 			(font
@@
 	(label "k02"
 		(at 29.21 60.96 0)
-		(fields_autoplaced yes)
 		(effects
 			(font
@@
 	(label "k03"
 		(at 29.21 58.42 0)
-		(fields_autoplaced yes)
 		(effects
 			(font
@@
 	(label "k10"
 		(at 29.21 93.98 0)
-		(fields_autoplaced yes)
 		(effects
 			(font
@@
 	(label "k13"
 		(at 180.34 73.66 0)
-		(fields_autoplaced yes)
 		(effects
 			(font
@@
 	(label "SCL"
 		(at 82.55 60.96 0)
-		(fields_autoplaced yes)
 		(effects
 			(font
@@
 	(label "k30"
 		(at 82.55 81.28 0)
-		(fields_autoplaced yes)
 		(effects
 			(font
@@
 	(label "k20"
 		(at 104.14 88.9 0)
-		(fields_autoplaced yes)
 		(effects
 			(font
@@
 	(label "k21"
 		(at 82.55 68.58 0)
-		(fields_autoplaced yes)
 		(effects
 			(font
@@
 	(label "k21"
 		(at 129.54 88.9 0)
-		(fields_autoplaced yes)
 		(effects
 			(font
@@
 	(label "k30"
 		(at 156.21 104.14 0)
-		(fields_autoplaced yes)
 		(effects
 			(font
@@
 	(label "TX"
 		(at 29.21 86.36 0)
-		(fields_autoplaced yes)
 		(effects
 			(font
@@
 	(label "k24"
 		(at 205.74 88.9 0)
-		(fields_autoplaced yes)
 		(effects
 			(font
@@
 	(label "k23"
 		(at 180.34 88.9 0)
-		(fields_autoplaced yes)
 		(effects
 			(font
@@
 	(label "k33"
 		(at 231.14 104.14 0)
-		(fields_autoplaced yes)
 		(effects
 			(font
@@
 	(label "k25"
 		(at 231.14 88.9 0)
-		(fields_autoplaced yes)
 		(effects
 			(font
@@
 	(label "k22"
 		(at 154.94 88.9 0)
-		(fields_autoplaced yes)
 		(effects
 			(font
@@
 	(label "k00"
 		(at 104.14 58.42 0)
-		(fields_autoplaced yes)
 		(effects
 			(font
@@
 	(label "TX"
 		(at 49.53 139.7 0)
-		(fields_autoplaced yes)
 		(effects
 			(font
@@
 	(label "k10"
 		(at 104.14 73.66 0)
-		(fields_autoplaced yes)
 		(effects
 			(font
@@
 	(label "k03"
 		(at 180.34 58.42 0)
-		(fields_autoplaced yes)
 		(effects
 			(font
@@
 	(label "RX"
 		(at 49.53 142.24 0)
-		(fields_autoplaced yes)
 		(effects
 			(font
@@
 	(label "k00"
 		(at 29.21 66.04 0)
-		(fields_autoplaced yes)
 		(effects
 			(font
@@
 	(label "k14"
 		(at 205.74 73.66 0)
-		(fields_autoplaced yes)
 		(effects
 			(font
@@
 	(label "k05"
 		(at 29.21 53.34 0)
-		(fields_autoplaced yes)
 		(effects
 			(font
@@
 	(label "k01"
 		(at 129.54 58.42 0)
-		(fields_autoplaced yes)
 		(effects
 			(font
@@
 	(label "k05"
 		(at 231.14 58.42 0)
-		(fields_autoplaced yes)
 		(effects
 			(font
@@
 	(label "k02"
 		(at 154.94 58.42 0)
-		(fields_autoplaced yes)
 		(effects
 			(font
@@
 	(label "k04"
 		(at 205.74 58.42 0)
-		(fields_autoplaced yes)
 		(effects
 			(font
@@
 	(label "k11"
 		(at 29.21 91.44 0)
-		(fields_autoplaced yes)
 		(effects
 			(font
@@
 	(label "k31"
 		(at 181.61 104.14 0)
-		(fields_autoplaced yes)
 		(effects
 			(font
@@
 	(label "SDA"
 		(at 29.21 78.74 0)
-		(fields_autoplaced yes)
 		(effects
 			(font
@@
 	(label "SDA"
 		(at 64.77 135.89 0)
-		(fields_autoplaced yes)
 		(effects
 			(font
@@
 	(label "k32"
 		(at 82.55 86.36 0)
-		(fields_autoplaced yes)
 		(effects
 			(font
@@
 	(label "k15"
 		(at 231.14 73.66 0)
-		(fields_autoplaced yes)
 		(effects
 			(font
@@
 	(label "k04"
 		(at 29.21 55.88 0)
-		(fields_autoplaced yes)
 		(effects
 			(font
@@
 			)
 		)
-		(property "Footprint" "YUKI:CherryMX_rev"
+		(property "Footprint" "YUKI:Kailh_Choc_PG1350_rev"
 			(at 167.64 73.66 0)
 			(effects
@@
 			)
 		)
-		(property "Footprint" "YUKI:CherryMX_rev"
+		(property "Footprint" "YUKI:Kailh_Choc_PG1350_rev"
 			(at 243.84 73.66 0)
 			(effects
@@
 			)
 		)
-		(property "Footprint" "YUKI:CherryMX_rev"
+		(property "Footprint" "YUKI:Kailh_Choc_PG1350_rev"
 			(at 243.84 104.14 0)
 			(effects
@@
 			)
 		)
-		(property "Footprint" "YUKI:CherryMX_rev"
+		(property "Footprint" "YUKI:Kailh_Choc_PG1350_rev"
 			(at 167.64 88.9 0)
 			(effects
@@
 			)
 		)
-		(property "Footprint" "YUKI:CherryMX_rev"
+		(property "Footprint" "YUKI:Kailh_Choc_PG1350_rev"
 			(at 218.44 88.9 0)
 			(effects
@@
 			)
 		)
-		(property "Footprint" "YUKI:CherryMX_rev"
+		(property "Footprint" "YUKI:Kailh_Choc_PG1350_rev"
 			(at 218.44 73.66 0)
 			(effects
@@
 			)
 		)
-		(property "Footprint" "YUKI:CherryMX_rev"
+		(property "Footprint" "YUKI:Kailh_Choc_PG1350_rev"
 			(at 243.84 88.9 0)
 			(effects
@@
 			)
 		)
-		(property "Footprint" "YUKI:CherryMX_rev"
+		(property "Footprint" "YUKI:Kailh_Choc_PG1350_rev"
 			(at 116.84 88.9 0)
 			(effects
@@
 			)
 		)
-		(property "Footprint" "YUKI:CherryMX_rev"
+		(property "Footprint" "YUKI:Kailh_Choc_PG1350_rev"
 			(at 218.44 58.42 0)
 			(effects
@@
 			)
 		)
-		(property "Footprint" "YUKI:CherryMX_rev"
+		(property "Footprint" "YUKI:Kailh_Choc_PG1350_rev"
 			(at 142.24 58.42 0)
 			(effects
@@
 			)
 		)
-		(property "Footprint" "YUKI:CherryMX_rev"
+		(property "Footprint" "YUKI:Kailh_Choc_PG1350_rev"
 			(at 243.84 58.42 0)
 			(effects
@@
 			)
 		)
-		(property "Footprint" "YUKI:CherryMX_rev"
+		(property "Footprint" "YUKI:Kailh_Choc_PG1350_rev"
 			(at 116.84 73.66 0)
 			(effects
@@
 			)
 		)
-		(property "Footprint" "YUKI:CherryMX_rev"
+		(property "Footprint" "YUKI:Kailh_Choc_PG1350_rev"
 			(at 142.24 73.66 0)
 			(effects
@@
 			)
 		)
-		(property "Footprint" "YUKI:CherryMX_rev"
+		(property "Footprint" "YUKI:Kailh_Choc_PG1350_rev"
 			(at 142.24 88.9 0)
 			(effects
@@
 			)
 		)
-		(property "Footprint" "YUKI:CherryMX_rev"
+		(property "Footprint" "YUKI:Kailh_Choc_PG1350_rev"
 			(at 194.31 104.14 0)
 			(effects
@@
 			)
 		)
-		(property "Footprint" "YUKI:CherryMX_rev"
+		(property "Footprint" "YUKI:Kailh_Choc_PG1350_rev"
 			(at 168.91 104.14 0)
 			(effects
@@
 			)
 		)
-		(property "Footprint" "YUKI:CherryMX_rev"
+		(property "Footprint" "YUKI:Kailh_Choc_PG1350_rev"
 			(at 193.04 58.42 0)
 			(effects
@@
 			)
 		)
-		(property "Footprint" "YUKI:CherryMX_rev"
+		(property "Footprint" "YUKI:Kailh_Choc_PG1350_rev"
 			(at 116.84 58.42 0)
 			(effects
@@
 			)
 		)
-		(property "Footprint" "YUKI:CherryMX_rev"
+		(property "Footprint" "YUKI:Kailh_Choc_PG1350_rev"
 			(at 193.04 73.66 0)
 			(effects
@@
 			)
 		)
-		(property "Footprint" "YUKI:CherryMX_rev"
+		(property "Footprint" "YUKI:Kailh_Choc_PG1350_rev"
 			(at 167.64 58.42 0)
 			(effects
@@
 			)
 		)
-		(property "Footprint" "YUKI:CherryMX_rev"
+		(property "Footprint" "YUKI:Kailh_Choc_PG1350_rev"
 			(at 219.71 104.14 0)
 			(effects
@@
 			)
 		)
-		(property "Footprint" "YUKI:CherryMX_rev"
+		(property "Footprint" "YUKI:Kailh_Choc_PG1350_rev"
 			(at 193.04 88.9 0)
 			(effects
